File: hw/goryn.kicad_pcb (KiCad board)
At the start: 2 copper layers, 50 x 50 mm, 53 parts, among them J1 Conn_FFC_30, J10 3V3, J2 Conn_FFC_30, J3 Conn_FFC_30, J30 EMI-shield-clip-corner, J31 EMI-shield-clip-corner, J32 EMI-shield-clip-corner, J33 EMI-shield-clip-corner, J4 Conn_FFC_30, J5 Conn_Coaxial, J6 USB_C_Receptacle_USB2.0_16P, J8 5V, J9 1V, U2 W25Q128JVS, U3 MT3520B, U4 MT3520B, X1 osc_4pin_3.2_2.5

Commit message: v1.0.0
Parts:
- removed J30, J31, J32, J33: EMI-shield-clip-corner, AI6YP:EMI-shield-clip-corner
- added C15: 22uF, AI6YP:C_0603_1608Metric, F.Cu at (87.0, 60.0)
- added H1: MountingHole_M3, AI6YP:MountingHole_3.2mm_M3_Pad_Via, F.Cu at (53.0, 97.0)
- added H2: MountingHole_M3, AI6YP:MountingHole_3.2mm_M3_Pad_Via, F.Cu at (97.0, 97.0)
- added H3: MountingHole_M3, AI6YP:MountingHole_3.2mm_M3_Pad_Via, F.Cu at (97.0, 53.0)
- added H4: MountingHole_M3, AI6YP:MountingHole_3.2mm_M3_Pad_Via, F.Cu at (53.0, 53.0)
- U1: footprint AI6YP:QFN-88-10x10mm-P0.4mm-EP6.74x6.74mm -> AI6YP:GIWIN-QFN-88-10x10mm-P0.4mm-EP6.74x6.74mm
- moved R2 19.2 mm to (96.0, 70.5), turned to -90 degrees
- moved R8 9.08 mm to (91.5, 54.0), turned to -90 degrees
- moved R7 7.14 mm to (89.5, 54.0), turned to -90 degrees
- moved R12 6.52 mm to (67.0, 95.0)
- moved R13 6.52 mm to (67.0, 96.5)
- moved R9 5.85 mm to (87.5, 54.0), turned to 90 degrees
- moved R42 5.15 mm to (98.0, 91.0), turned to 90 degrees
- moved U2 3.89 mm to (93.0, 59.9)
- moved C31 3.35 mm to (60.5, 95.5)
- moved R10 3.17 mm to (55.0, 81.0)
- moved R11 3.17 mm to (53.5, 81.0)
- moved J6 2.59 mm to (52.3, 89.0)
- moved J5 1.58 mm to (53.5, 58.5)
- moved R41 1.12 mm to (96.0, 91.0)
- moved R14 0.71 mm to (60.0, 62.0)
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Connections:
- net MSPI_CLK renamed /East/IOR34_N
- net MSPI_CS renamed /East/IOR34_P
- net MSPI_DI renamed /East/IOR33_N
- net MSPI_DO renamed /East/IOR33_P
- net MSPI_HOLD renamed /East/IOR29A
- net MSPI_WP renamed /East/IOR35A
Routing:
- net /East/IOR34_N: track 48.9 -> 32.9 mm, vias 0 -> 2
- net Net-(J6-D--PadA7): track 7.77 -> 20.2 mm
- net Net-(J6-D+-PadA6): track 9.32 -> 20.6 mm
- net +3V3: track 150.6 -> 159.8 mm, vias 14 -> 15
- net /South/IOB6_P: track 23.4 -> 16.6 mm
- net /South/IOB6_N: track 23.6 -> 18.3 mm
- net /East/IOR33_N: track 33.1 -> 28.8 mm
- net +5V: track 15.9 -> 18.3 mm, vias 8 -> 7
- net /East/IOR33_P: track 31.0 -> 28.7 mm
- net /East/IOR29A: track 32.6 -> 30.3 mm
- net Net-(J6-CC1): track 6.88 -> 8.94 mm
- net /East/IOR34_P: track 32.7 -> 34.7 mm, vias 2 -> 0
- net /East/IOR35A: track 43.2 -> 41.9 mm, vias 2 -> 0
- net Net-(U4-FB): track 4.92 -> 5.94 mm
- net GND: track 2.40 -> 1.47 mm, vias 178 -> 191
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Other:
- outline, holes or cut-outs redrawn
